File: small-board/tms-rgb.sch (EAGLE design)
At the start: 39 parts, among them J1 Pads, U1 CD74HC4053PWR, U100 TMS992XA, U2 TS5A4597DCKR, U3 LM1881MX/NOPB, U4 MAX4395EUD, U5 SN74LVC2G17DCKR, U6 LMH1251MT/NOPB, U7 THS7374IPWR

Commit message: Nudged C4 on the schematic
It's the sample-and-hold cap but its position (near the SPST instead of the op-amp) didn't reflect that clearly.
Other:
- note added: "Nicholas Piegdon May 17, 2020 v1+ CERN-OHL-W v2 github.com/npiegdon/tms-rgb nicholas.piegdon.info/tms-rgb @npiegdon"
- note removed: "Nicholas Piegdon May 17, 2020 v1 CERN-OHL-W v2 github.com/npiegdon/tms-rgb nicholas.piegdon.info/tms-rgb @npiegdon"
- moved on the sheet: C10, C11, C12, C13, C14, C15, C16, C2, C3, C4, C5, C6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
